File: ergogen/output/pcbs/frontplate.kicad_pcb (KiCad board)
At the start: 2 copper layers, 133.3 x 91.7 mm, 0 parts

Commit message: Refresh generated files.
Parts:
- added H1: , Screw_Hole, F.Cu at (109.5, 71.5)
- added H2: , Screw_Hole, F.Cu at (109.5, 90.5)
- added H3: , Screw_Hole, F.Cu at (185.5, 68.0)
- added H4: , Screw_Hole, F.Cu at (152.7, 107.7)
- added H5: , Screw_Hole, F.Cu at (199.2, 115.3)
Changed lines of the file:
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@@
     (add_net "")
+  )
+  (module "Screw_Hole" (layer F.Cu)
+      (at 109.5 71.5 0)
+      (fp_text reference "H1" (at 0 2.55) (layer F.SilkS) hide (effects (font (size 1 1) (thickness 0.15))))
+      (pad "" np_thru_hole circle (at 0 0) (size 2.2 2.2) (drill 2.2) (layers *.Cu *.Mask))
+  )
+  (module "Screw_Hole" (layer F.Cu)
+      (at 109.5 90.5 0)
+      (fp_text reference "H2" (at 0 2.55) (layer F.SilkS) hide (effects (font (size 1 1) (thickness 0.15))))
+      (pad "" np_thru_hole circle (at 0 0) (size 2.2 2.2) (drill 2.2) (layers *.Cu *.Mask))
+  )
+  (module "Screw_Hole" (layer F.Cu)
+      (at 185.468 67.986 0)
+      (fp_text reference "H3" (at 0 2.55) (layer F.SilkS) hide (effects (font (size 1 1) (thickness 0.15))))
+      (pad "" np_thru_hole circle (at 0 0) (size 2.2 2.2) (drill 2.2) (layers *.Cu *.Mask))
+  )
+  (module "Screw_Hole" (layer F.Cu)
+      (at 152.657 107.74 0)
+      (fp_text reference "H4" (at 0 2.55) (layer F.SilkS) hide (effects (font (size 1 1) (thickness 0.15))))
+      (pad "" np_thru_hole circle (at 0 0) (size 2.2 2.2) (drill 2.2) (layers *.Cu *.Mask))
+  )
+  (module "Screw_Hole" (layer F.Cu)
+      (at 199.2410516 115.3236576 60)
+      (fp_text reference "H5" (at 0 2.55) (layer F.SilkS) hide (effects (font (size 1 1) (thickness 0.15))))
+      (pad "" np_thru_hole circle (at 0 0) (size 2.2 2.2) (drill 2.2) (layers *.Cu *.Mask))
   )
             (gr_line (start 91.08198222285509 108.74001780012622) (end 91.08001777794281 53.49000464193523) (angle 90) (layer Edge.Cuts) (width 0.15))
