File: ergogen/output/pcbs/corney_island_mx_partially_routed.kicad_pcb (KiCad board)
At the start: 2 copper layers, 133.8 x 91.7 mm, 94 parts

Commit message: Update assets
Routing:
- net GND: track 101.4 -> 183.3 mm, vias 27 -> 39
- net C5: track 91.4 -> 169.5 mm
- net C3: track 213.3 -> 277.2 mm
- net C4: track 91.4 -> 155.2 mm
- net VCC: track 101.4 -> 150.8 mm, vias 27 -> 33
- net C2: track 68.6 -> 106.6 mm
- net C0: track 190.5 -> 228.5 mm
- net C1: track 68.6 -> 106.6 mm
- net R0: track 112.1 -> 147.1 mm
- net R2: track 112.1 -> 147.1 mm
- net R1: track 112.1 -> 147.1 mm
- net R3: track 56.1 -> 80.7 mm
- net ULED_6: track 13.5 -> 24.8 mm
- net ULED_5: track 13.5 -> 24.8 mm
- net ULED_4: track 13.5 -> 24.8 mm
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