File: ergogen/output/pcbs/corney_island_mx_partially_routed.kicad_pcb (KiCad board)
At the start: 2 copper layers, 133.8 x 91.7 mm, 94 parts

Commit message: Update assets
Parts:
- removed B1: Reset (PTS636 SP43 LFS), ceoloide:top-actuated-reset-switch
- removed DISP1: , combo_display
- removed LED1, LED10, LED11, LED12, LED13, LED14, LED15, LED16, LED17, LED18, LED19, LED2, LED20, LED21, LED3, LED4, LED5, LED6, LED7, LED8, LED9: , ceoloide:YS-SK6812MINI-E (per-key)
- removed LED22, LED23, LED24, LED25, LED26, LED27: , ceoloide:YS-SK6812MINI-E (underglow)
- removed TRRS1: TRRS-PJ-320A-dual, TRRS-PJ-320A-dual
Connections:
- MCU1 pad 119: P3 -> SCL
- MCU1 pad 120: P2 -> SDA
Routing:
- net VCC: track 150.8 -> 49.4 mm, vias 33 -> 6
- net GND: track 183.3 -> 81.9 mm, vias 39 -> 12
- net (no net): track 0.00 -> 67.9 mm
- net ULED_6: track 24.8 -> 0.00 mm, vias 2 -> 0
- net ULED_5: track 24.8 -> 0.00 mm, vias 2 -> 0
- net ULED_4: track 24.8 -> 0.00 mm, vias 2 -> 0
- net ULED_3: track 24.8 -> 0.00 mm, vias 2 -> 0
- net ULED_2: track 24.8 -> 0.00 mm, vias 2 -> 0
- net LED_1: track 24.8 -> 0.00 mm, vias 2 -> 0
- net LED_3: track 13.5 -> 0.00 mm, vias 2 -> 0
- net LED_4: track 13.5 -> 0.00 mm, vias 2 -> 0
- net LED_8: track 13.5 -> 0.00 mm, vias 2 -> 0
- net LED_7: track 13.5 -> 0.00 mm, vias 2 -> 0
- net LED_6: track 13.5 -> 0.00 mm, vias 2 -> 0
- net LED_20: track 13.5 -> 0.00 mm, vias 2 -> 0
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Other:
- outline, holes or cut-outs redrawn
