File: ergogen/output/pcbs/corney_island_autorouted.kicad_pcb (KiCad board)
At the start: 2 copper layers, 133.8 x 91.7 mm, 94 parts

Commit message: Update assets
Routing:
- net C5: track 205.0 -> 165.7 mm, vias 4 -> 6
- net LED_16: track 58.1 -> 36.6 mm, vias 3 -> 2
- net GND: track 657.8 -> 636.6 mm, vias 41 -> 27
- net ULED_1: track 55.8 -> 36.6 mm, vias 5 -> 2
- net SCL: track 47.0 -> 28.6 mm, vias 0 -> 1
- net VCC: track 663.0 -> 644.6 mm, vias 39 -> 28
- net mid_home: track 22.5 -> 40.6 mm, vias 1 -> 2
- net R2: track 184.7 -> 202.0 mm, vias 7 -> 8
- net C0: track 243.5 -> 258.8 mm, vias 3 -> 4
- net C2: track 205.3 -> 192.7 mm, vias 4 -> 3
- net R1: track 170.7 -> 182.4 mm, vias 6 -> 8
- net R0: track 181.4 -> 192.2 mm, vias 6 -> 8
- net R3: track 137.2 -> 127.0 mm
- net LED_9: track 55.1 -> 45.7 mm
- net LED_11: track 49.5 -> 40.4 mm
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
Commit message: Update assets
Routing:
- net LED_17: track 40.9 -> 90.3 mm, vias 4 -> 3
- net R0: track 192.2 -> 230.1 mm, vias 8 -> 4
- net C5: track 165.7 -> 201.0 mm, vias 6 -> 3
- net VCC: track 644.6 -> 678.9 mm, vias 28 -> 29
- net C0: track 258.8 -> 237.8 mm, vias 4 -> 2
- net R3: track 127.0 -> 146.5 mm
- net C1: track 229.2 -> 210.2 mm
- net mid_home: track 40.6 -> 21.8 mm, vias 2 -> 1
- net R2: track 202.0 -> 220.4 mm, vias 8 -> 7
- net R1: track 182.4 -> 198.9 mm, vias 8 -> 7
- net GND: track 636.6 -> 622.9 mm, vias 27 -> 29
- net SDA: track 19.6 -> 32.2 mm, vias 1 -> 0
- net C4: track 200.8 -> 212.9 mm, vias 5 -> 4
- net LED_1: track 22.8 -> 33.4 mm, vias 3 -> 2
- net ULED_2: track 21.2 -> 30.4 mm
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
Commit message: Update assets
Routing:
- net LED_17: track 90.3 -> 47.8 mm, vias 3 -> 2
- net R2: track 220.4 -> 194.8 mm, vias 7 -> 9
- net DAT: track 57.6 -> 81.0 mm
- net C5: track 201.0 -> 184.4 mm
- net R0: track 230.1 -> 245.5 mm, vias 4 -> 3
- net C1: track 210.2 -> 224.7 mm, vias 4 -> 1
- net C3: track 228.2 -> 218.5 mm
- net ULED_3: track 31.5 -> 21.9 mm
- net ULED_2: track 30.4 -> 22.5 mm
- net ULED_4: track 28.9 -> 21.3 mm, vias 2 -> 3
- net VCC: track 678.9 -> 671.5 mm
- net LED_14: track 48.9 -> 42.0 mm
- net C4: track 212.9 -> 219.7 mm, vias 4 -> 3
- net ULED_5: track 29.2 -> 22.6 mm, vias 2 -> 3
- net LED_16: track 45.2 -> 38.7 mm, vias 5 -> 2
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
Commit message: Update assets
Parts:
- TRRS1: footprint TRRS-PJ-320A-dual -> ceoloide:TRRS-PJ-320A-dual (reversible, symmetric)
- moved LED22 78.9 mm to (195.0, 69.1)
- moved LED24 49.0 mm to (119.0, 71.5)
- moved LED25 46.1 mm to (119.0, 90.5)
- moved LED23 38.7 mm to (157.0, 64.4)
- moved LED26 38.3 mm to (157.0, 102.4)
- moved LED27 38.0 mm to (195.0, 107.1)
Connections:
- LED1 pad 2: LED_19 -> LED_21
- LED1 pad 4: LED_18 -> LED_20
- LED10 pad 2: ULED_4 -> LED_10
- LED10 pad 4: LED_10 -> LED_9
- LED11 pad 2: LED_10 -> LED_11
- LED11 pad 4: LED_9 -> LED_10
- LED12 pad 2: ULED_3 -> LED_12
- LED12 pad 4: LED_8 -> LED_11
- LED13 pad 2: LED_6 -> LED_7
- LED13 pad 4: LED_5 -> LED_6
- LED14 pad 2: LED_7 -> LED_6
- LED14 pad 4: LED_6 -> LED_5
- LED15 pad 2: LED_8 -> LED_5
- LED15 pad 4: LED_7 -> LED_4
- LED16 pad 2: ULED_2 -> LED_2
- LED16 pad 4: LED_2 -> LED_1
- LED17 pad 2: LED_2 -> LED_3
- LED17 pad 4: ULED_1 -> LED_2
- LED18 pad 2: LED_1 -> LED_4
- LED18 pad 4: LED -> LED_3
- LED19 pad 2: LED_12 -> LED_9
- LED19 pad 4: LED_11 -> LED_8
- LED20 pad 2: LED_5 -> LED_8
- LED20 pad 4: LED_4 -> LED_7
- LED21 pad 2: LED_4 -> LED_1
- LED21 pad 4: LED_3 -> ULED_6
- LED22 pad 2: LED_17 -> ULED_1
- LED22 pad 4: ULED_6 -> LED
- LED23 pad 2: LED_16 -> ULED_2
- LED23 pad 4: ULED_5 -> ULED_1
- LED24 pad 2: LED_11 -> ULED_3
- LED24 pad 4: ULED_4 -> ULED_2
- LED25 pad 2: LED_9 -> ULED_4
- LED26 pad 2: LED_3 -> ULED_5
- LED26 pad 4: ULED_2 -> ULED_4
- LED27 pad 2: ULED_1 -> ULED_6
- LED27 pad 4: LED_1 -> ULED_5
- LED3 pad 2: LED_21 -> LED_19
- LED3 pad 4: LED_20 -> LED_18
- LED4 pad 2: LED_18 -> LED_16
- LED4 pad 4: LED_17 -> LED_15
- LED5 pad 2: ULED_6 -> LED_17
- LED6 pad 2: ULED_5 -> LED_18
- LED6 pad 4: LED_15 -> LED_17
- LED7 pad 2: LED_13 -> LED_15
- LED7 pad 4: LED_12 -> LED_14
- LED9 pad 2: LED_15 -> LED_13
- LED9 pad 4: LED_14 -> LED_12
- MCU1 pad 119: P3 -> SCL
- MCU1 pad 120: P2 -> SDA
- TRRS1 pad 2: DAT -> GND
- TRRS1 pad 3: GND -> VCC
Routing:
- net R0: track 245.5 -> 176.0 mm, vias 3 -> 7
- net ULED_4: track 21.3 -> 83.4 mm, vias 3 -> 5
- net VCC: track 671.5 -> 628.8 mm, vias 29 -> 32
- net ULED_5: track 22.6 -> 62.3 mm
- net C4: track 219.7 -> 184.6 mm, vias 3 -> 4
- net LED_7: track 51.5 -> 80.9 mm, vias 2 -> 5
- net C5: track 184.4 -> 157.7 mm, vias 3 -> 4
- net DAT: track 81.0 -> 54.4 mm
- net R1: track 195.4 -> 170.1 mm, vias 8 -> 10
- net ULED_3: track 21.9 -> 47.0 mm, vias 3 -> 2
- net ULED_6: track 28.5 -> 53.3 mm, vias 2 -> 3
- net LED_1: track 28.8 -> 51.2 mm
- net LED: track 29.7 -> 51.9 mm, vias 2 -> 1
- net ULED_2: track 22.5 -> 44.6 mm, vias 3 -> 2
- net LED_12: track 40.9 -> 22.9 mm
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Other:
- outline, holes or cut-outs redrawn

Commit message: Update assets
Parts:
- LED1, LED10, LED11, LED12, LED13, LED14, LED15, LED16, LED17, LED18, LED19, LED2, LED20, LED21, LED3, LED4, LED5, LED6, LED7, LED8, LED9: footprint ceoloide:YS-SK6812MINI-E (per-key) -> ceoloide:YS-SK6812MINI-E (per-key, reversible)
- LED22, LED23, LED24, LED25, LED26, LED27: footprint ceoloide:YS-SK6812MINI-E (underglow) -> ceoloide:YS-SK6812MINI-E (underglow, reversible)
Routing:
- net C3: track 236.3 -> 200.5 mm, vias 7 -> 4
- net C2: track 185.5 -> 220.6 mm, vias 4 -> 3
- net GND: track 623.6 -> 647.3 mm, vias 32 -> 30
- net LED_7: track 80.9 -> 61.6 mm, vias 5 -> 3
- net R2: track 195.2 -> 176.4 mm
- net R3: track 133.4 -> 151.0 mm
- net LED: track 51.9 -> 34.7 mm, vias 1 -> 2
- net VCC: track 628.8 -> 643.2 mm, vias 32 -> 36
- net R1: track 170.1 -> 180.6 mm
- net SDA: track 41.1 -> 49.1 mm
- net C1: track 242.4 -> 235.0 mm, vias 3 -> 7
- net C0: track 244.9 -> 251.9 mm, vias 6 -> 3
- net C4: track 184.6 -> 179.1 mm, vias 4 -> 5
- net LED_16: track 49.0 -> 43.5 mm
- net ULED_6: track 53.3 -> 58.3 mm
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Other:
- outline, holes or cut-outs redrawn
- net class Default removed

Commit message: Update assets
Routing:
- net C2: track 220.6 -> 194.1 mm, vias 3 -> 5
- net VCC: track 643.2 -> 623.0 mm
- net GND: track 647.3 -> 627.4 mm, vias 30 -> 32
- net C0: track 251.9 -> 270.3 mm
- net LED: track 34.7 -> 51.9 mm, vias 2 -> 1
- net C5: track 160.1 -> 173.2 mm, vias 5 -> 6
- net R1: track 180.6 -> 167.9 mm, vias 10 -> 11
- net LED_7: track 61.6 -> 74.0 mm, vias 3 -> 4
- net C1: track 235.0 -> 245.7 mm, vias 7 -> 3
- net SCL: track 33.9 -> 44.3 mm, vias 1 -> 2
- net C3: track 200.5 -> 209.9 mm, vias 4 -> 5
- net ULED_6: track 58.3 -> 49.2 mm, vias 3 -> 4
- net SDA: track 49.1 -> 41.2 mm
- net LED_3: track 47.4 -> 41.6 mm
- net R3: track 151.0 -> 145.2 mm, vias 6 -> 3
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Other:
- outline, holes or cut-outs redrawn
- net class Default added: clearance 0.2, trace_width 0.25, via_dia 0.8, via_drill 0.4

Commit message: Update assets
Parts:
- added MH1: , ceoloide:mounting_hole_npth, F.Cu at (207.8, 100.5)
- added MH2: , ceoloide:mounting_hole_npth, F.Cu at (222.2, 109.0)
- added MH3: , ceoloide:mounting_hole_npth, F.Cu at (109.5, 71.5)
- added MH4: , ceoloide:mounting_hole_npth, F.Cu at (109.5, 90.5)
- added MH5: , ceoloide:mounting_hole_npth, F.Cu at (185.5, 68.0)
- added MH6: , ceoloide:mounting_hole_npth, F.Cu at (152.7, 107.7)
- added MH7: , ceoloide:mounting_hole_npth, F.Cu at (199.2, 115.3)
- D1, D10, D11, D12, D13, D14, D15, D16, D17, D18, D19, D2, D20, D21, D22, D23, D24, D25, D26, D27, D28, D29, D3, D30, D31, D32, D33, D34, D35, D36, D37, D38, D39, D4, D40, D41, D42, D5, D6, D7, D8, D9: footprint ComboDiode -> ceoloide:diode_tht_sod123
- DISP1: footprint combo_display -> ceoloide:display_ssd1306_nice_view
- LED1, LED10, LED11, LED12, LED13, LED14, LED15, LED16, LED17, LED18, LED19, LED2, LED20, LED21, LED3, LED4, LED5, LED6, LED7, LED8, LED9: footprint ceoloide:YS-SK6812MINI-E (per-key, reversible) -> ceoloide:led_SK6812mini-e (per-key, reversible)
- LED22, LED23, LED24, LED25, LED26, LED27: footprint ceoloide:YS-SK6812MINI-E (underglow, reversible) -> ceoloide:led_SK6812mini-e (underglow, reversible)
- MCU1: footprint nice_nano -> ceoloide:nice_nano
- RST1: renamed from B1; value Reset (PTS636 SP43 LFS) -> reset_switch_tht_top; footprint ceoloide:top-actuated-reset-switch -> ceoloide:reset_switch_tht_top
- TRRS1: footprint ceoloide:TRRS-PJ-320A-dual (reversible, symmetric) -> ceoloide:trrs_pj320a (reversible, symmetric)
- moved D20 0.40 mm to (195.0, 118.3)
- moved D41 0.40 mm to (180.7, 114.4)
- moved D1 0.40 mm to (107.4, 98.7)
- moved D10 0.40 mm to (164.4, 91.5)
- moved D11 0.40 mm to (164.4, 72.5)
- moved D12 0.40 mm to (164.4, 53.5)
- moved D13 0.40 mm to (183.4, 93.9)
- moved D14 0.40 mm to (183.4, 74.9)
- moved D15 0.40 mm to (183.4, 55.9)
- moved D16 0.40 mm to (202.4, 96.3)
- moved D17 0.40 mm to (202.4, 77.3)
- moved D18 0.40 mm to (202.4, 58.3)
- moved D19 0.40 mm to (173.9, 113.5)
- moved D2 0.40 mm to (107.4, 79.7)
- moved D22 0.40 mm to (92.6, 98.7)
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Connections:
- MCU1 pad 13: MCU1_13 -> MCU1_12
- MCU1 pad 14: MCU1_14 -> MCU1_11
- MCU1 pad 15: MCU1_15 -> MCU1_10
- MCU1 pad 16: MCU1_16 -> MCU1_9
- MCU1 pad 17: MCU1_17 -> MCU1_8
- MCU1 pad 18: MCU1_18 -> MCU1_7
- MCU1 pad 19: MCU1_19 -> MCU1_6
- MCU1 pad 20: MCU1_20 -> MCU1_5
- MCU1 pad 21: MCU1_21 -> MCU1_4
- MCU1 pad 22: MCU1_22 -> MCU1_3
- MCU1 pad 23: MCU1_23 -> MCU1_2
- MCU1 pad 24: MCU1_24 -> MCU1_1
- TRRS1 pad 3: VCC -> DAT
Routing:
- net C0: track 270.3 -> 241.1 mm, vias 3 -> 1
- net C1: track 245.7 -> 217.7 mm
- net GND: track 627.4 -> 655.2 mm, vias 32 -> 28
- net VCC: track 623.0 -> 647.1 mm, vias 36 -> 33
- net ULED_4: track 85.5 -> 64.2 mm, vias 5 -> 3
- net LED: track 51.9 -> 34.3 mm, vias 1 -> 2
- net R0: track 179.7 -> 167.1 mm
- net R2: track 181.9 -> 170.9 mm, vias 9 -> 7
- net SCL: track 44.3 -> 33.3 mm, vias 2 -> 1
- net R1: track 167.9 -> 178.8 mm, vias 11 -> 8
- net C5: track 173.2 -> 163.9 mm
- net LED_6: track 45.1 -> 53.4 mm, vias 4 -> 3
- net DAT: track 54.6 -> 62.1 mm
- net R3: track 145.2 -> 137.8 mm, vias 3 -> 4
- net C4: track 178.5 -> 185.1 mm, vias 5 -> 7
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Other:
- outline, holes or cut-outs redrawn
- net class Default removed

Commit message: Update assets
Parts:
- DISP1: footprint ceoloide:display_ssd1306_nice_view -> ceoloide:display_ssd1306
- MCU1: footprint ceoloide:nice_nano -> ceoloide:mcu_nice_nano
- moved DISP1 14.6 mm to (214.6, 76.6)
Connections:
- DISP1 pad 11: DISP1_4 -> DISP1_2
- DISP1 pad 13: DISP1_2 -> DISP1_4
- DISP1 pad 14: DISP1_1 -> GND
- DISP1 pad 21: DISP1_4 -> DISP1_3
- DISP1 pad 22: DISP1_3 -> DISP1_2
- DISP1 pad 23: DISP1_2 -> DISP1_1
- DISP1 pad 24: DISP1_1 -> GND
Routing:
- net R2: track 170.9 -> 211.7 mm
- net ULED_4: track 64.2 -> 89.7 mm, vias 3 -> 5
- net R1: track 178.8 -> 155.3 mm, vias 8 -> 9
- net C4: track 185.1 -> 197.4 mm, vias 7 -> 5
- net C1: track 217.7 -> 227.0 mm, vias 3 -> 5
- net LED_6: track 53.4 -> 45.9 mm, vias 3 -> 2
- net middle_home: track 23.4 -> 30.6 mm
- net LED_11: track 47.7 -> 41.7 mm, vias 2 -> 3
- net LED_5: track 41.6 -> 45.9 mm, vias 3 -> 2
- net SDA: track 47.4 -> 43.2 mm
- net R3: track 137.8 -> 141.7 mm, vias 4 -> 5
- net C5: track 163.9 -> 160.1 mm
- net DISP1_4: track 0.00 -> 3.50 mm
- net DISP1_3: track 0.00 -> 3.50 mm
- net DISP1_2: track 0.00 -> 3.50 mm
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