File: ergogen/output/pcbs/corney_island_autorouted.kicad_pcb (KiCad board)
At the start: 2 copper layers, 133.8 x 91.7 mm, 122 parts

Commit message: Update assets
Routing:
- net GND: track 130.3 -> 662.5 mm, vias 27 -> 31
- net VCC: track 111.0 -> 634.8 mm, vias 27 -> 33
- net C0: track 9.64 -> 238.7 mm, vias 0 -> 2
- net C1: track 9.64 -> 210.5 mm, vias 0 -> 5
- net R2: track 9.63 -> 203.3 mm, vias 0 -> 6
- net C3: track 9.64 -> 198.5 mm, vias 0 -> 4
- net C2: track 9.64 -> 192.3 mm, vias 0 -> 4
- net C4: track 9.64 -> 181.9 mm, vias 0 -> 5
- net C5: track 9.64 -> 166.5 mm, vias 0 -> 4
- net R1: track 9.63 -> 166.4 mm, vias 0 -> 7
- net R0: track 9.63 -> 165.7 mm, vias 0 -> 8
- net R3: track 9.63 -> 138.5 mm, vias 0 -> 4
- net ULED_4: track 13.5 -> 85.1 mm, vias 2 -> 4
- net LED_7: track 13.5 -> 74.9 mm, vias 2 -> 4
- net DAT: track 9.63 -> 57.0 mm
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