File: ergogen/output/pcbs/corney_island_wireless.kicad_pcb (KiCad board)
At the start: 2 copper layers, 133.8 x 91.7 mm, 75 parts

Commit message: Update footprints library and artifacts
Connections:
- MCU1 pad 1: RAW -> LED
- MCU1 pad 10: C5 -> R2
- MCU1 pad 11: P16 -> R3
- MCU1 pad 113: P9 -> P10
- MCU1 pad 114: R3 -> P16
- MCU1 pad 115: R2 -> C5
- MCU1 pad 116: R1 -> C4
- MCU1 pad 117: R0 -> C3
- MCU1 pad 118: CS -> C2
- MCU1 pad 119: SCL -> C1
- MCU1 pad 12: P10 -> P9
- MCU1 pad 120: SDA -> C0
- MCU1 pad 121: GND -> VCC
- MCU1 pad 122: GND -> RST
- MCU1 pad 123: DAT -> GND
- MCU1 pad 124: LED -> RAW
- MCU1 pad 2: GND -> DAT
- MCU1 pad 3: RST -> GND
- MCU1 pad 4: VCC -> GND
- MCU1 pad 5: C0 -> SDA
- MCU1 pad 6: C1 -> SCL
- MCU1 pad 7: C2 -> CS
- MCU1 pad 8: C3 -> R0
- MCU1 pad 9: C4 -> R1
