File: filtered-output/pcbs/cad/left_pcb.kicad_pcb (KiCad board)
At the start: 2 copper layers, 132.6 x 134.8 mm, 137 parts

Commit message: updated outputs
Parts:
- added H1, H2: , ceoloide:header-preview_nano, F.Cu at (81.8, 47.8)
- added SC1: , ceoloide:screw-preview-top, F.Cu at (41.8, 85.4)
- added SC10: , ceoloide:screw-preview-bottom, F.Cu at (131.7, 156.4)
- added SC2: , ceoloide:screw-preview-top, F.Cu at (41.8, 136.4)
- added SC3: , ceoloide:screw-preview-top, F.Cu at (126.8, 80.1)
- added SC4: , ceoloide:screw-preview-top, F.Cu at (126.8, 131.1)
- added SC5: , ceoloide:screw-preview-top, F.Cu at (131.7, 156.4)
- added SC6: , ceoloide:screw-preview-bottom, F.Cu at (41.8, 85.4)
- added SC7: , ceoloide:screw-preview-bottom, F.Cu at (41.8, 136.4)
- added SC8: , ceoloide:screw-preview-bottom, F.Cu at (126.8, 80.1)
- added SC9: , ceoloide:screw-preview-bottom, F.Cu at (126.8, 131.1)
- added ST1: , ceoloide:standoff-preview, F.Cu at (41.8, 85.4)
- added ST2: , ceoloide:standoff-preview, F.Cu at (41.8, 136.4)
- added ST3: , ceoloide:standoff-preview, F.Cu at (126.8, 80.1)
- added ST4: , ceoloide:standoff-preview, F.Cu at (126.8, 131.1)
- added ST5: , ceoloide:standoff-preview, F.Cu at (131.7, 156.4)
- moved MH5 13.0 mm to (131.7, 156.4)
- moved MH3 13.0 mm to (126.8, 80.1)
- moved MH4 13.0 mm to (126.8, 131.1)
- moved MH1 13.0 mm to (41.8, 85.4)
- moved MH2 13.0 mm to (41.8, 136.4)
