File: filtered-output/pcbs/cad/right_pcb.kicad_pcb (KiCad board)
At the start: 2 copper layers, 132.6 x 134.8 mm, 132 parts

Commit message: updated outputs
Parts:
- added H1, H2: , ceoloide:header-preview_nano, F.Cu at (255.2, 47.8)
